Commit message: Enhance RRT and RRT* planners with collision checking and pathfinding improvements
- Refactored RRTPlanner to include detailed collision checking, goal biasing, and path reconstruction.
- Introduced RRTStarPlanner with radius-based rewiring and improved cost calculations for optimal pathfinding.
- Added unit tests for A* planner utilities, ensuring correct world-to-cell conversions and inflation behavior.
- Updated CMakeLists.txt to install helper scripts for robot description publishing.
- Enhanced RViz configuration for better visualization of occupancy and planned paths.
- Modified bringup launch file to include inflation radius as a parameter and improved robot spawning logic.
- Streamlined smoke test script for headless operation, focusing on essential topic checks and logging.

File: src/robot_maze_description/urdf/maze_generate/lidar.urdf.xacro (robot description, xacro)
@@ -42,26 +42,29 @@
         </joint>
         <gazebo reference="${child}_link">
-            <material>Gazebo/Black</material>
-            <sensor name="laser" type="gpu_lidar">
-                <pose> 0 0 0 0 0 0 </pose>
-                <always_on>true</always_on>
-                <visualize>true</visualize>
-                <update_rate>10</update_rate>
-                <topic>lidarscan</topic>
-                <gz_frame_id>${child}_link</gz_frame_id>
-                <lidar>
-                    <scan>
-                        <horizontal>
-                            <samples>360</samples>
-                            <min_angle>-3.14</min_angle>
-                            <max_angle>3.14</max_angle>
-                        </horizontal>
-                    </scan>
-                    <range>
-                        <min>0.15</min>
-                        <max>12</max>
-                    </range>
-                </lidar>
-            </sensor>
+        <sensor name="laser" type="gpu_lidar">
+            <pose>0 0 0 0 0 0</pose>
+            <update_rate>10</update_rate>
+            <visualize>true</visualize>
+            <topic>/scan</topic> <lidar>
+            <scan>
+                <horizontal>
+                <samples>360</samples>
+                <min_angle>-3.14</min_angle>
+                <max_angle>3.14</max_angle>
+                </horizontal>
+            </scan>
+            <range>
+                <min>0.15</min>
+                <max>12.0</max>
+            </range>
+            </lidar>
+            <plugin filename="libgz-sim-laserscan-system.so"
+                    name="gz::sim::systems::LaserScan">
+            <ros>
+                <namespace></namespace>
+                <topic>/scan</topic> <frame_id>${child}_link</frame_id>
+            </ros>
+            </plugin>
+        </sensor>
         </gazebo>
     </xacro:macro>
